File: elec/layout/default/ah3772-sa-7.kicad_pcb (KiCad board)
At the start: 2 copper layers, 225.7 x 100.8 mm, 0 parts

Commit message: layout
Parts:
- added C1: 16V 100nF X7R ±10% 0402 Multilayer Ceramic Capacitors MLCC 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, lib:C0402, F.Cu at (162.1, 86.0)
- added R1: Chip Resistor - Surface Mount 1KOhms ±5% 1/16W 0402 RoHS, lib:R0402, F.Cu at (162.3, 81.6)
- added U1: , lib:SOT-23-3_L2.9-W1.3-P1.90-LS2.4-BR-CW, F.Cu at (161.9, 83.8)
Routing:
- net vcc: track 0.00 -> 6.54 mm
- net out: track 0.00 -> 1.38 mm
Changed lines of the file:
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@@
   )
   (net 0 "")
+  (net 1 "gnd")
+  (net 2 "out")
+  (net 3 "vcc")
+  (footprint "lib:R0402" (layer "F.Cu")
+    (at 162.254297 81.643967)
+    (descr "Resistor SMD 0402 (1005 Metric), square (rectangular) end terminal, IPC_7351 nominal, (Body size source: IPC-SM-782 page 72, https://www.pcb-3d.com/wordpress/wp-content/uploads/ipc-sm-782a_amendment_1_and_2.pdf), generated with kicad-footprint-generator")
+    (tags "resistor")
+    (attr smd)
+    (fp_text reference "R1" (at 0 -1.17) (layer "F.SilkS")
+        (effects (font (size 1 1) (thickness 0.15)))
+    )
+    (fp_text value "Chip Resistor - Surface Mount 1KOhms ±5% 1/16W 0402 RoHS" (at 0 1.17) (layer "F.Fab")
+        (effects (font (size 1 1) (thickness 0.15)))
+    )
+    (fp_text user "${REFERENCE}" (at 0 0) (layer "F.Fab")
+        (effects (font (size 0.26 0.26) (thickness 0.04)))
+    )
+    (fp_line (start -0.153641 -0.38) (end 0.153641 -0.38)
+      (stroke (width 0.12) (type solid)) (layer "F.SilkS"))
+    (fp_line (start -0.153641 0.38) (end 0.153641 0.38)
+      (stroke (width 0.12) (type solid)) (layer "F.SilkS"))
+    (fp_line (start -0.93 -0.47) (end 0.93 -0.47)
+      (stroke (width 0.05) (type solid)) (layer "F.CrtYd"))
+    (fp_line (start -0.93 0.47) (end -0.93 -0.47)
+      (stroke (width 0.05) (type solid)) (layer "F.CrtYd"))
+    (fp_line (start 0.93 -0.47) (end 0.93 0.47)
+      (stroke (width 0.05) (type solid)) (layer "F.CrtYd"))
+    (fp_line (start 0.93 0.47) (end -0.93 0.47)
+      (stroke (width 0.05) (type solid)) (layer "F.CrtYd"))
+    (fp_line (start -0.525 -0.27) (end 0.525 -0.27)
+      (stroke (width 0.1) (type solid)) (layer "F.Fab"))
+    (fp_line (start -0.525 0.27) (end -0.525 -0.27)
+      (stroke (width 0.1) (type solid)) (layer "F.Fab"))
+    (fp_line (start 0.525 -0.27) (end 0.525 0.27)
+      (stroke (width 0.1) (type solid)) (layer "F.Fab"))
+    (fp_line (start 0.525 0.27) (end -0.525 0.27)
+      (stroke (width 0.1) (type solid)) (layer "F.Fab"))
+    (pad "1" smd roundrect (at -0.51 0) (size 0.54 0.64) (layers "F.Cu" "F.Paste" "F.Mask") (roundrect_rratio 0.25)
+      (net 3 "vcc") (pintype "stereo"))
+    (pad "2" smd roundrect (at 0.51 0) (size 0.54 0.64) (layers "F.Cu" "F.Paste" "F.Mask") (roundrect_rratio 0.25)
+      (net 2 "out") (pintype "stereo"))
+    (model "${KICAD6_3DMODEL_DIR}/Resistor_SMD.3dshapes/R_0402_1005Metric.wrl"
+      (offset (xyz 0 0 0))
+      (scale (xyz 1 1 1))
+      (rotate (xyz 0 0 0))
+    )
+  )
+  (footprint "lib:SOT-23-3_L2.9-W1.3-P1.90-LS2.4-BR-CW" (layer "F.Cu")
+    (at 161.87 83.83)
+    (attr through_hole)
+    (fp_text reference "U1" (at 0 -4.95) (layer "F.SilkS")
+        (effects (font (size 1 1) (thickness 0.15)))
+    )
+    (fp_text value "" (at 0 4.95) (layer "F.Fab")
+        (effects (font (size 1 1) (thickness 0.15)))
+    )
+    (fp_text user "${REFERENCE}" (at 0 0) (layer "F.Fab")
+        (effects (font (size 1 1) (thickness 0.15)))
+    )
+    (fp_line (start -0.65 -1.46) (end -0.65 -0.8)
+      (stroke (width 0.25) (type solid)) (layer "F.SilkS"))
+    (fp_line (start -0.65 -1.46) (end 0.17 -1.46)
+      (stroke (width 0.25) (type solid)) (layer "F.SilkS"))
+    (fp_line (start -0.65 -0.8) (end -0.65 -1.46)
+      (stroke (width 0.25) (type solid)) (layer "F.SilkS"))
+    (fp_line (start -0.65 -0.8) (end -0.65 -1.46)
+      (stroke (width 0.25) (type solid)) (layer "F.SilkS"))
+    (fp_line (start -0.65 1.46) (end -0.65 0.8)
+      (stroke (width 0.25) (type solid)) (layer "F.SilkS"))
+    (fp_line (start 0.17 1.46) (end -0.65 1.46)
+      (stroke (width 0.25) (type solid)) (layer "F.SilkS"))
+    (fp_line (start 0.76 0.3) (end 0.76 -0.3)
+      (stroke (width 0.2) (type solid)) (layer "F.SilkS"))
+    (fp_circle (center 1.27 1.02) (end 1.4 1.02)
+      (stroke (width 0.25) (type solid)) (fill none) (layer "Cmts.User"))
+    (fp_circle (center 1.2 1.45) (end 1.23 1.45)
+      (stroke (width 0.06) (type solid)) (fill none) (layer "F.Fab"))
+    (pad "1" smd rect (at 1.25 0.95) (size 1.15 0.7) (layers "F.Cu" "F.Paste" "F.Mask")
+      (net 3 "vcc") (pintype "stereo"))
+    (pad "2" smd rect (at -1.25 0) (size 1.15 0.7) (layers "F.Cu" "F.Paste" "F.Mask")
+      (net 1 "gnd") (pintype "stereo"))
+    (pad "3" smd rect (at 1.25 -0.95) (size 1.15 0.7) (layers "F.Cu" "F.Paste" "F.Mask")
+      (net 2 "out") (pintype "stereo"))
+    (model "/Users/narayanpowderly/Documents/atopile-workspace/swoop/.ato/modules/ah3772-sa-7/elec/footprints/footprints.3dshapes/SOT-23-3_L2.9-W1.3-P1.90-LS2.4-BR-CW.wrl"
+      (offset (xyz 0 -0 0))
+      (scale (xyz 1 1 1))
+      (rotate (xyz 0 0 0))
+    )
+  )
+  (footprint "lib:C0402" (layer "F.Cu")
+    (at 162.135535 86.013842)
+    (descr "Capacitor SMD 0402 (1005 Metric), square (rectangular) end terminal, IPC_7351 nominal, (Body size source: IPC-SM-782 page 76, https://www.pcb-3d.com/wordpress/wp-content/uploads/ipc-sm-782a_amendment_1_and_2.pdf), generated with kicad-footprint-generator")
+    (tags "capacitor")
+    (attr smd)
+    (fp_text reference "C1" (at 0 -1.16) (layer "F.SilkS")
+        (effects (font (size 1 1) (thickness 0.15)))
+    )
+    (fp_text value "16V 100nF X7R ±10% 0402  Multilayer Ceramic Capacitors MLCC - SMD/SMT ROHS" (at 0 1.16) (layer "F.Fab")
+        (effects (font (size 1 1) (thickness 0.15)))
+    )
+    (fp_text user "${REFERENCE}" (at 0 0) (layer "F.Fab")
+        (effects (font (size 0.25 0.25) (thickness 0.04)))
+    )
+    (fp_line (start -0.107836 -0.36) (end 0.107836 -0.36)
+      (stroke (width 0.12) (type solid)) (layer "F.SilkS"))
+    (fp_line (start -0.107836 0.36) (end 0.107836 0.36)
+      (stroke (width 0.12) (type solid)) (layer "F.SilkS"))
+    (fp_line (start -0.91 -0.46) (end 0.91 -0.46)
+      (stroke (width 0.05) (type solid)) (layer "F.CrtYd"))
+    (fp_line (start -0.91 0.46) (end -0.91 -0.46)
+      (stroke (width 0.05) (type solid)) (layer "F.CrtYd"))
+    (fp_line (start 0.91 -0.46) (end 0.91 0.46)
+      (stroke (width 0.05) (type solid)) (layer "F.CrtYd"))
+    (fp_line (start 0.91 0.46) (end -0.91 0.46)
+      (stroke (width 0.05) (type solid)) (layer "F.CrtYd"))
+    (fp_line (start -0.5 -0.25) (end 0.5 -0.25)
+      (stroke (width 0.1) (type solid)) (layer "F.Fab"))
+    (fp_line (start -0.5 0.25) (end -0.5 -0.25)
+      (stroke (width 0.1) (type solid)) (layer "F.Fab"))
+    (fp_line (start 0.5 -0.25) (end 0.5 0.25)
+      (stroke (width 0.1) (type solid)) (layer "F.Fab"))
+    (fp_line (start 0.5 0.25) (end -0.5 0.25)
+      (stroke (width 0.1) (type solid)) (layer "F.Fab"))
+    (pad "1" smd roundrect (at -0.48 0) (size 0.56 0.62) (layers "F.Cu" "F.Paste" "F.Mask") (roundrect_rratio 0.25)
+      (net 3 "vcc") (pintype "stereo"))
+    (pad "2" smd roundrect (at 0.48 0) (size 0.56 0.62) (layers "F.Cu" "F.Paste" "F.Mask") (roundrect_rratio 0.25)
+      (net 1 "gnd") (pintype "stereo"))
+    (model "${KICAD6_3DMODEL_DIR}/Capacitor_SMD.3dshapes/C_0402_1005Metric.wrl"
+      (offset (xyz 0 0 0))
+      (scale (xyz 1 1 1))
+      (rotate (xyz 0 0 0))
+    )
+  )
   (gr_circle (center 225.62 81.79) (end 227.32 81.79)
     (stroke (width 0.1) (type solid)) (fill none) (layer "Edge.Cuts"))
@@
       (xy 69.100734 49.778315)
     )
-    (stroke (width 0) (type solid)) (fill none) (layer "Edge.Cuts"))
+    (stroke (width 0.1) (type solid)) (fill none) (layer "Edge.Cuts"))
   (gr_arc (start 261.62 113.79) (mid 260.448427 116.618427) (end 257.62 117.79)
     (stroke (width 0.1) (type solid)) (layer "Edge.Cuts"))
@@
     (effects (font (size 2 2) (thickness 0.1)) (justify left bottom))
   )
+  (segment (start 162.764297 82.524297) (end 163.12 82.88) (width 0.25) (layer "F.Cu") (net 2))
+  (segment (start 162.764297 81.643967) (end 162.764297 82.524297) (width 0.25) (layer "F.Cu") (net 2))
+  (segment (start 161.655535 85.419465) (end 162.295 84.78) (width 0.25) (layer "F.Cu") (net 3))
+  (segment (start 162.295 84.78) (end 163.12 84.78) (width 0.25) (layer "F.Cu") (net 3))
+  (segment (start 161.655535 86.013842) (end 161.655535 85.419465) (width 0.25) (layer "F.Cu") (net 3))
+  (segment (start 161.744297 84.268629) (end 161.744297 81.643967) (width 0.25) (layer "F.Cu") (net 3))
+  (segment (start 163.12 84.78) (end 162.255668 84.78) (width 0.25) (layer "F.Cu") (net 3))
+  (segment (start 162.255668 84.78) (end 161.744297 84.268629) (width 0.25) (layer "F.Cu") (net 3))
   (group "" (id 6c1ef9f7-0f34-47bb-ac1a-76df23fb396e)
     (members
