File: elec/layout/default/ah3772-sa-7.kicad_pcb (KiCad board)
At the start: 2 copper layers, 225.7 x 100.8 mm, 3 parts

Commit message: update layout
Parts:
- R1: value Chip Resistor - Surface Mount 1KOhms ±5% 1/16W 0402 RoHS -> 62.5mW Thick Film Resistors ±100ppm/℃ ±1% 1kΩ 0402 Chip Resistor - Surface Mount ROHS
Changed lines of the file:
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@@
         (effects (font (size 1 1) (thickness 0.15)))
     )
-    (fp_text value "Chip Resistor - Surface Mount 1KOhms ±5% 1/16W 0402 RoHS" (at 0 1.17) (layer "F.Fab")
+    (fp_text value "62.5mW Thick Film Resistors ±100ppm/℃ ±1% 1kΩ 0402  Chip Resistor - Surface Mount ROHS" (at 0 1.17) (layer "F.Fab")
         (effects (font (size 1 1) (thickness 0.15)))
     )
